File: Board Files/PicoPad.sch (KiCad schematic (older format))
At the start: 23 parts, among them U1 CD4021BE, U2 SW_Push

Commit message: Add labels to schematic
Parts:
- U1: value CD4021BE -> CD4021BPW
Other:
- note added: "BUTTONS\n"
- note added: "CABLE CONNECTIONS\n\n"
- note added: "PULL-UP RESISTORS\n"
- note added: "SHIFT REGISTER\n"
Changed lines of the file:
@@
 EESchema Schematic File Version 4
-LIBS:PicoPad-cache
 EELAYER 29 0
 EELAYER END
@@
 P 6050 3350
 F 0 "U1" H 6050 4320 50  0000 C CNN
-F 1 "CD4021BE" H 6050 4229 50  0000 C CNN
+F 1 "CD4021BPW" H 6050 4229 50  0000 C CNN
 F 2 "Package_SO:TSSOP-16_4.4x5mm_P0.65mm" H 6050 3350 50  0001 L BNN
 F 3 "" H 6050 3350 50  0001 L BNN
@@
 Text Label 7450 3500 1    50   ~ 0
 GND
+Wire Notes Line
+	5250 1400 5250 2050
+Wire Notes Line
+	5250 2050 7200 2050
+Wire Notes Line
+	7200 2050 7200 1400
+Wire Notes Line
+	7200 1400 5250 1400
+Text Notes 5800 1350 0    50   ~ 0
+CABLE CONNECTIONS\n\n
+Text Notes 2800 1750 0    50   ~ 0
+PULL-UP RESISTORS\n
+Text Notes 5700 4700 0    50   ~ 0
+SHIFT REGISTER\n
+Text Notes 2200 5050 0    50   ~ 0
+BUTTONS\n
 $EndSCHEMATC
